File: UINIO-MCU-ESP32S3.kicad_pcb (KiCad board)
At the start: 2 copper layers, 91.1 x 20.3 mm, 52 parts, among them J1 Conn_01x03_Pin, J2 Conn_01x27_Pin, J3 Conn_01x04_Pin, J4 Conn_01x27_Pin, SW1 复位, SW2 启动选择, U1 ME6211C33M5G-N, U2 W25Q128JVSSIQ, U3 ESP-PSRAM64H, U4 RS2227XUTQK10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

Commit message: Complete PCB wiring.
Parts:
- moved C14 54.0 mm to (126.7, 109.1)
- moved C1 53.7 mm to (115.9, 108.4)
- moved C10 53.7 mm to (177.3, 107.7)
- moved C15 53.7 mm to (181.9, 110.0)
- moved C16 53.7 mm to (181.9, 111.7)
- moved C8 53.7 mm to (182.5, 107.0)
- moved C9 53.7 mm to (179.1, 107.7)
- moved L1 53.7 mm to (183.9, 106.6)
- moved R6 53.7 mm to (174.8, 111.4)
- moved SW1 53.7 mm to (138.7, 110.3)
- moved SW2 53.7 mm to (138.7, 105.1)
- moved U1 53.7 mm to (116.3, 106.0)
- moved U2 53.7 mm to (146.6, 107.7)
- moved U6 53.7 mm to (129.7, 109.3)
- moved ? 53.7 mm to (112.7, 107.9)
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Routing:
- net /VDD_3.3V: track 56.9 -> 206.6 mm, vias 2 -> 12
- net GND: track 36.1 -> 128.2 mm, vias 1 -> 104
- net /GPIO0: track 35.9 -> 68.7 mm, vias 0 -> 2
- net /VDD_5V: track 29.5 -> 56.0 mm, vias 3 -> 4
- net /CHIP_PU: track 56.8 -> 81.8 mm, vias 2 -> 6
- net /SPICLK/GPIO30: track 40.0 -> 62.7 mm
- net /DTR: track 18.4 -> 41.0 mm, vias 1 -> 5
- net /SPICS1/GPIO26: track 43.5 -> 62.1 mm, vias 1 -> 0
- net /SPID/GPIO32: track 33.4 -> 52.0 mm
- net /SPICS0/GPIO29: track 30.0 -> 38.9 mm, vias 0 -> 1
- net /SPIQ/GPIO31: track 37.1 -> 42.4 mm
- net /USB_Data+: track 14.7 -> 11.5 mm
- net /GPIO10: track 13.9 -> 15.3 mm
- net /SPIWP/GPIO28: track 45.1 -> 43.8 mm, vias 1 -> 0
- net Net-(U5-XTAL_N): track 12.0 -> 11.3 mm
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- added copper zone on B.Cu, net GND
- added copper zone on F.Cu, net GND
Other:
- outline, holes or cut-outs redrawn
- board text added: "下载方式"
- board text added: "可选项"
- board text removed: "下载选择"
- board text removed: "可选装"

Commit message: Complete PCB wiring.
Parts:
- moved SW1 0.06 mm to (138.6, 110.4)
- turned C3 to -90 degrees
- turned C4 to -90 degrees
- turned C6 to -90 degrees
Routing:
- net GND: track 128.2 -> 132.5 mm, vias 104 -> 126
- net /VDD_3.3V: track 206.6 -> 204.8 mm

Commit message: Complete PCB wiring.
Parts:
- added ?: LOGO, LOGO, B.Cu at (149.5, 107.6)
Routing:
- net /DTR: track 41.0 -> 39.5 mm
Other:
- board text added: "Tensilica Xtensa LX"
- board text added: "UINIO-MCU-ESP32S3"
- board text added: "Version 1.0.0"

Commit message: update PCB.
Parts:
- moved ? 1.24 mm to (148.3, 107.5)
Routing:
- net GND: track 132.5 -> 156.1 mm, vias 126 -> 147
- net /SPIHD/GPIO27: track 46.7 -> 69.0 mm, vias 0 -> 3
- net /SPIWP/GPIO28: track 43.8 -> 60.1 mm, vias 0 -> 1
- net /GPIO45: track 3.94 -> 12.2 mm, vias 0 -> 2
- net /VDD_3.3V: track 204.8 -> 210.2 mm, vias 12 -> 13
Other:
- board text added: "G0"
- board text added: "G1"
- board text added: "G10"
- board text added: "G11"
- board text added: "G12"
- board text added: "G13"
- board text added: "G14"
- board text added: "G15"
- board text added: "G16"
- board text added: "G17"
- board text added: "G18"
- board text added: "G19"
- board text added: "G2"
- board text added: "G20"
- board text added: "G21"
- board text added: "G26"
- board text added: "G27"
- board text added: "G28"
- board text added: "G29"
- board text added: "G3"
- board text added: "G30"
- board text added: "G31"
- board text added: "G32"
- board text added: "G33"
- board text added: "G34"
- board text added: "G35"
- board text added: "G36"
- board text added: "G37"
- board text added: "G39"
- board text added: "G4"
- board text added: "G40"
- board text added: "G41"
- board text added: "G42"
- board text added: "G45"
- board text added: "G46"
- board text added: "G47"
- board text added: "G48"
- board text added: "G5"
- board text added: "G6"
- board text added: "G7"
- board text added: "G8"
- board text added: "G9"
- board text added: "Tensilica Xtensa LX7"
- board text added: "可留空"
- board text removed: "IO0"
- board text removed: "IO1"
- board text removed: "IO10"
- board text removed: "IO11"
- board text removed: "IO12"
- board text removed: "IO13"
- board text removed: "IO14"
- board text removed: "IO15"
- board text removed: "IO16"
- board text removed: "IO17"
- board text removed: "IO18"
- board text removed: "IO19"
- board text removed: "IO2"
- board text removed: "IO20"
- board text removed: "IO21"
- board text removed: "IO26"
- board text removed: "IO27"
- board text removed: "IO28"
- board text removed: "IO29"
- board text removed: "IO3"
- board text removed: "IO30"
- board text removed: "IO31"
- board text removed: "IO32"
- board text removed: "IO33"
- board text removed: "IO34"
- board text removed: "IO35"
- board text removed: "IO36"
- board text removed: "IO37"
- board text removed: "IO39"
- board text removed: "IO4"
- board text removed: "IO40"
- board text removed: "IO41"
- board text removed: "IO42"
- board text removed: "IO45"
- board text removed: "IO46"
- board text removed: "IO47"
- board text removed: "IO48"
- board text removed: "IO5"
- board text removed: "IO6"
- board text removed: "IO7"
- board text removed: "IO8"
- board text removed: "IO9"
- board text removed: "Tensilica Xtensa LX"
- board text removed: "可选项"

Commit message: update PCB.
Parts:
- moved ? 0.39 mm to (148.6, 107.3)
Routing:
- net GND: vias 147 -> 149

Commit message: Update PCB.
Routing:
- net GND: track 156.1 -> 161.7 mm, vias 149 -> 147
- net Net-(AE1-FEED): track 0.87 -> 5.62 mm
- net /USB_Data+: track 11.5 -> 14.7 mm

Commit message: Update PCB.
Other:
- board text added: "SPICLK"
- board text added: "SPICS0"
- board text added: "SPICS1"
- board text added: "SPIHD"
- board text added: "SPIQ"
- board text added: "SPIWP"
- board text added: "VDDSPI"
- board text added: "可选"
- board text removed: "G26"
- board text removed: "G27"
- board text removed: "G28"
- board text removed: "G29"
- board text removed: "G30"
- board text removed: "G31"
- board text removed: "可留空"

Commit message: Update PCB.
Parts:
- moved ? 20.8 mm to (167.2, 98.0)
- moved AE1 9.72 mm to (188.9, 93.5)
- moved C1 9.72 mm to (116.1, 98.7)
- moved C10 9.72 mm to (177.5, 98.0)
- moved C11 9.72 mm to (121.6, 98.3)
- moved C15 9.72 mm to (182.2, 100.3)
- moved C16 9.72 mm to (182.2, 102.0)
- moved C19 9.72 mm to (173.9, 101.7)
- moved C3 9.72 mm to (177.5, 95.4)
- moved C4 9.72 mm to (179.3, 95.4)
- moved C6 9.72 mm to (181.2, 95.4)
- moved C8 9.72 mm to (182.7, 97.3)
- moved C9 9.72 mm to (179.3, 98.0)
- moved L1 9.72 mm to (184.1, 96.8)
- moved R6 9.72 mm to (175.1, 101.7)
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Routing:
- net GND: track 161.7 -> 164.6 mm
- net Net-(AE1-FEED): track 5.62 -> 6.55 mm
Other:
- outline, holes or cut-outs redrawn
- board text added: "Candence"
- board text added: "Tensilica Xtensa Dual-Core LX7"
- board text removed: "Tensilica Xtensa LX7"
