File: UINIO-MCU-ESP32S3.kicad_pcb (KiCad board)
At the start: 2 copper layers, 87.4 x 20.3 mm, 48 parts, among them J1 Conn_01x03_Pin, J2 Conn_01x27_Pin, J3 Conn_01x04_Pin, J4 Conn_01x27_Pin, SW1 复位, SW2 启动选择, U1 ME6211C33M5G-N, U2 W25Q128JVSSIQ, U3 ESP-PSRAM64H, U4 RS2227XUTQK10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

Commit message: Release UINIO-MCU-ESP32S3 version 3.5.0.
Parts:
- moved C10 1.34 mm to (175.7, 98.5)
- moved C9 1.33 mm to (178.4, 98.5)
- moved C6 0.43 mm to (181.6, 94.5)
- moved C19 0.38 mm to (173.6, 101.9)
- moved R6 0.38 mm to (174.8, 101.9)
- moved C7 0.23 mm to (177.9, 92.8)
- moved R4 0.23 mm to (181.1, 92.8)
- moved C4 0.22 mm to (179.6, 94.5)
Routing:
- net GND: track 199.9 -> 181.2 mm, vias 149 -> 157
- net /VDD_3.3V: track 239.2 -> 236.8 mm
- net /GPIO10: track 15.3 -> 14.3 mm
- net /GPIO45: track 12.2 -> 11.3 mm, vias 2 -> 0

Commit message: Release UINIO-MCU-ESP32S3 version 3.5.0.
Routing:
- net GND: track 181.2 -> 186.0 mm, vias 157 -> 164

Commit message: Release UINIO-MCU-ESP32S3 version 3.5.0.
Parts:
- moved C7 0.14 mm to (177.9, 92.9)
- moved R4 0.14 mm to (181.1, 92.9)
