File: UINIO-MCU-ESP32S3.kicad_sch (KiCad schematic)
At the start: 47 parts, among them J1 Conn_01x03_Pin, J2 Conn_01x27_Pin, J3 Conn_01x04_Pin, J4 Conn_01x27_Pin, SW1 复位, SW2 启动选择, U1 ME6211C33M5G-N, U2 W25Q128JVSSIQ, U3 ESP-PSRAM64H, U4 RS2227XUTQK10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

Commit message: Release UINIO-MCU-ESP32S3 version 3.1.1.
Other:
- company: 电子技术博客 UinIO.com -> UinIO.com 电子技术实验室
Changed lines of the file:
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@@
   (title_block
     (title "UINIO-MCU-ESP32S3")
-    (date "2023-07-06")
-    (rev "Version 3.1.0")
-    (company "电子技术博客 UinIO.com")
+    (date "2024-01-10")
+    (rev "Version 3.1.1")
+    (company "UinIO.com 电子技术实验室")
   )
   (junction (at 91.44 228.6) (diameter 0) (color 0 0 0 0)

Commit message: Update PCB layout.
Parts:
- removed C5, C8: TBD, Capacitor_SMD:C_0402_1005Metric, symbol Device:C
- removed L1: TBD, Inductor_SMD:L_0402_1005Metric, symbol Device:L
Connections:
- net at AE1.1 (FEED): now also U5.1 (LNA_IN)
Other:
- moved on the sheet: AE1
Changed lines of the file:
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@@
   (title_block
     (title "UINIO-MCU-ESP32S3")
-    (date "2024-01-31")
-    (rev "Version 3.2.1")
+    (date "2024-03-05")
+    (rev "Version 3.3.0")
     (company "UinIO.com 电子技术实验室")
   )
@@
   (junction (at 341.63 161.29) (diameter 0) (color 0 0 0 0)
   )
-  (junction (at 158.75 67.31) (diameter 0) (color 0 0 0 0)
-  )
   (junction (at 196.85 231.14) (diameter 0) (color 0 0 0 0)
   )
@@
   (junction (at 260.35 113.03) (diameter 0) (color 0 0 0 0)
   )
-  (junction (at 171.45 67.31) (diameter 0) (color 0 0 0 0)
-  )
   (junction (at 203.2 55.88) (diameter 0) (color 0 0 0 0)
   )
@@
     (stroke (width 0) (type default))
   )
-  (wire (pts (xy 158.75 74.93) (xy 158.75 76.2))
-    (stroke (width 0) (type default))
-  )
   (wire (pts (xy 325.12 53.34) (xy 323.85 53.34))
     (stroke (width 0) (type default))
@@
     (stroke (width 0) (type default))
   )
-  (wire (pts (xy 158.75 67.31) (xy 161.29 67.31))
-    (stroke (width 0) (type default))
-  )
   (wire (pts (xy 142.24 123.19) (xy 142.24 124.46))
     (stroke (width 0) (type default))
@@
     (stroke (width 0) (type default))
   )
-  (wire (pts (xy 171.45 67.31) (xy 168.91 67.31))
-    (stroke (width 0) (type default))
-  )
   (wire (pts (xy 215.9 64.77) (xy 215.9 52.07))
     (stroke (width 0) (type default))
@@
     (stroke (width 0) (type default))
   )
-  (wire (pts (xy 142.24 67.31) (xy 142.24 68.58))
+  (wire (pts (xy 152.4 72.39) (xy 152.4 73.66))
     (stroke (width 0) (type default))
   )
@@
     (stroke (width 0) (type default))
   )
-  (wire (pts (xy 171.45 74.93) (xy 171.45 76.2))
-    (stroke (width 0) (type default))
-  )
   (wire (pts (xy 242.57 39.37) (xy 255.27 39.37))
     (stroke (width 0) (type default))
@@
     (stroke (width 0) (type default))
   )
-  (wire (pts (xy 184.15 80.01) (xy 187.96 80.01))
+  (wire (pts (xy 157.48 80.01) (xy 187.96 80.01))
     (stroke (width 0) (type default))
   )
@@
     (stroke (width 0) (type default))
   )
-  (wire (pts (xy 184.15 67.31) (xy 184.15 80.01))
+  (wire (pts (xy 157.48 72.39) (xy 157.48 80.01))
     (stroke (width 0) (type default))
   )
@@
     (stroke (width 0) (type default))
   )
-  (wire (pts (xy 171.45 67.31) (xy 184.15 67.31))
-    (stroke (width 0) (type default))
-  )
   (wire (pts (xy 196.85 231.14) (xy 201.93 231.14))
     (stroke (width 0) (type default))
@@
     (stroke (width 0) (type default))
   )
-  (wire (pts (xy 147.32 67.31) (xy 158.75 67.31))
-    (stroke (width 0) (type default))
-  )
   (wire (pts (xy 88.9 93.98) (xy 104.14 93.98))
     (stroke (width 0) (type default))
@@
     )
   )
-  (symbol (lib_id "power:GND") (at 171.45 76.2 0) (unit 1)
+  (symbol (lib_id "power:GND") (at 152.4 73.66 0) (unit 1)
     (in_bom yes) (on_board yes) (dnp no)
-    (property "Reference" "#PWR017" (at 171.45 82.55 0)
+    (property "Reference" "#PWR011" (at 152.4 80.01 0)
       (effects (font (size 1.27 1.27)) hide)
     )
-    (property "Value" "GND" (at 171.45 80.01 0)
+    (property "Value" "GND" (at 152.4 77.47 0)
       (effects (font (size 1.27 1.27)))
     )
-    (property "Footprint" "" (at 171.45 76.2 0)
+    (property "Footprint" "" (at 152.4 73.66 0)
       (effects (font (size 1.27 1.27)) hide)
     )
-    (property "Datasheet" "" (at 171.45 76.2 0)
-      (effects (font (size 1.27 1.27)) hide)
-    )
-    (pin "1")
-    (instances
-      (project "UINIO-MCU-ESP32S3"
-        (path "/7b5dffae-532b-44bd-828e-e231478b308d"
-          (reference "#PWR017") (unit 1)
-        )
-      )
-    )
-  )
-  (symbol (lib_id "power:GND") (at 142.24 68.58 0) (unit 1)
-    (in_bom yes) (on_board yes) (dnp no)
-    (property "Reference" "#PWR011" (at 142.24 74.93 0)
-      (effects (font (size 1.27 1.27)) hide)
-    )
-    (property "Value" "GND" (at 142.24 72.39 0)
-      (effects (font (size 1.27 1.27)))
-    )
-    (property "Footprint" "" (at 142.24 68.58 0)
-      (effects (font (size 1.27 1.27)) hide)
-    )
-    (property "Datasheet" "" (at 142.24 68.58 0)
+    (property "Datasheet" "" (at 152.4 73.66 0)
       (effects (font (size 1.27 1.27)) hide)
     )
@@
     )
   )
-  (symbol (lib_id "Device:Antenna_Chip") (at 144.78 64.77 0) (mirror y) (unit 1)
+  (symbol (lib_id "Device:Antenna_Chip") (at 154.94 69.85 0) (mirror y) (unit 1)
     (in_bom yes) (on_board yes) (dnp no)
-    (property "Reference" "AE1" (at 140.335 56.515 0)
+    (property "Reference" "AE1" (at 150.495 61.595 0)
       (effects (font (size 1.27 1.27)) (justify right))
     )
-    (property "Value" "Antenna_Chip" (at 143.51 60.96 0)
+    (property "Value" "Antenna_Chip" (at 153.67 66.04 0)
       (effects (font (size 1.27 1.27)) (justify right))
     )
-    (property "Footprint" "RF_Antenna:Texas_SWRA117D_2.4GHz_Right" (at 147.32 60.325 0)
+    (property "Footprint" "RF_Antenna:Texas_SWRA117D_2.4GHz_Right" (at 157.48 65.405 0)
       (effects (font (size 1.27 1.27)) hide)
     )
-    (property "Datasheet" "~" (at 147.32 60.325 0)
+    (property "Datasheet" "~" (at 157.48 65.405 0)
       (effects (font (size 1.27 1.27)) hide)
     )
@@
     )
   )
-  (symbol (lib_id "Device:C") (at 158.75 71.12 0) (unit 1)
-    (in_bom yes) (on_board yes) (dnp no)
-    (property "Reference" "C5" (at 161.29 71.12 0)
-      (effects (font (size 1.27 1.27)) (justify left))
-    )
-    (property "Value" "TBD" (at 158.75 73.66 0)
-      (effects (font (size 1.27 1.27)) (justify left))
-    )
-    (property "Footprint" "Capacitor_SMD:C_0402_1005Metric" (at 159.7152 74.93 0)
-      (effects (font (size 1.27 1.27)) hide)
-    )
-    (property "Datasheet" "~" (at 158.75 71.12 0)
-      (effects (font (size 1.27 1.27)) hide)
-    )
-    (pin "1")
-    (pin "2")
-    (instances
-      (project "UINIO-MCU-ESP32S3"
-        (path "/7b5dffae-532b-44bd-828e-e231478b308d"
-          (reference "C5") (unit 1)
-        )
-      )
-    )
-  )
   (symbol (lib_id "power:GND") (at 368.3 30.48 270) (unit 1)
     (in_bom yes) (on_board yes) (dnp no)
@@
     )
   )
-  (symbol (lib_id "Device:C") (at 171.45 71.12 0) (unit 1)
-    (in_bom yes) (on_board yes) (dnp no)
-    (property "Reference" "C8" (at 173.99 71.12 0)
-      (effects (font (size 1.27 1.27)) (justify left))
-    )
-    (property "Value" "TBD" (at 171.45 73.66 0)
-      (effects (font (size 1.27 1.27)) (justify left))
-    )
-    (property "Footprint" "Capacitor_SMD:C_0402_1005Metric" (at 172.4152 74.93 0)
-      (effects (font (size 1.27 1.27)) hide)
-    )
-    (property "Datasheet" "~" (at 171.45 71.12 0)
-      (effects (font (size 1.27 1.27)) hide)
-    )
-    (pin "1")
-    (pin "2")
-    (instances
-      (project "UINIO-MCU-ESP32S3"
-        (path "/7b5dffae-532b-44bd-828e-e231478b308d"
-          (reference "C8") (unit 1)
-        )
-      )
-    )
-  )
   (symbol (lib_id "power:GND") (at 81.28 231.14 90) (unit 1)
     (in_bom yes) (on_board yes) (dnp no)
@@
     )
   )
-  (symbol (lib_id "Device:L") (at 165.1 67.31 90) (unit 1)
-    (in_bom yes) (on_board yes) (dnp no)
-    (property "Reference" "L1" (at 168.91 64.77 90)
-      (effects (font (size 1.27 1.27)))
-    )
-    (property "Value" "TBD" (at 162.56 64.77 90)
-      (effects (font (size 1.27 1.27)))
-    )
-    (property "Footprint" "Inductor_SMD:L_0402_1005Metric" (at 165.1 67.31 0)
-      (effects (font (size 1.27 1.27)) hide)
-    )
-    (property "Datasheet" "~" (at 165.1 67.31 0)
-      (effects (font (size 1.27 1.27)) hide)
-    )
-    (pin "1")
-    (pin "2")
-    (instances
-      (project "UINIO-MCU-ESP32S3"
-        (path "/7b5dffae-532b-44bd-828e-e231478b308d"
-          (reference "L1") (unit 1)
-        )
-      )
-    )
-  )
   (symbol (lib_id "power:GND") (at 43.18 157.48 270) (unit 1)
     (in_bom yes) (on_board yes) (dnp no)
@@
         )
       )
-    )
-  )
-  (symbol (lib_id "power:GND") (at 158.75 76.2 0) (unit 1)
-    (in_bom yes) (on_board yes) (dnp no)
-    (property "Reference" "#PWR015" (at 158.75 82.55 0)
-      (effects (font (size 1.27 1.27)) hide)
-    )
-    (property "Value" "GND" (at 158.75 80.01 0)
-      (effects (font (size 1.27 1.27)))
-    )
-    (property "Footprint" "" (at 158.75 76.2 0)
-      (effects (font (size 1.27 1.27)) hide)
-    )
-    (property "Datasheet" "" (at 158.75 76.2 0)
-      (effects (font (size 1.27 1.27)) hide)
-    )
-    (pin "1")
-    (instances
-      (project "UINIO-MCU-ESP32S3"
-        (path "/7b5dffae-532b-44bd-828e-e231478b308d"
-          (reference "#PWR015") (unit 1)
-        )
-      )

Commit message: Release UINIO-MCU-ESP32S3 version 3.5.0.
Parts:
- removed AE1: Antenna_Chip, RF_Antenna:Texas_SWRA117D_2.4GHz_Right, symbol Device:Antenna_Chip
- added L1: AN9520-245, Uinio:ANT-SMD_L9.5-W2.1, symbol Uinio:AN9520-245
Connections:
- net at U5.1 (LNA_IN): now also L1.1
- no-connect marks 8 -> 9
Changed lines of the file:
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@@
   (title_block
     (title "UINIO-MCU-ESP32S3")
-    (date "2024-03-05")
-    (rev "Version 3.3.0")
+    (date "2024-03-30")
+    (rev "Version 3.5.0")
     (company "UinIO.com 电子技术实验室")
   )
@@
   (no_connect (at 289.56 231.14))
   (no_connect (at 289.56 223.52))
+  (no_connect (at 149.86 63.5))
   (no_connect (at 289.56 233.68))
   (no_connect (at 71.12 223.52))
@@
     (stroke (width 0) (type default))
   )
+  (wire (pts (xy 149.86 63.5) (xy 149.86 66.04))
+    (stroke (width 0) (type default))
+  )
   (wire (pts (xy 379.73 76.2) (xy 381 76.2))
     (stroke (width 0) (type default))
@@
     (stroke (width 0) (type default))
   )
-  (wire (pts (xy 152.4 72.39) (xy 152.4 73.66))
-    (stroke (width 0) (type default))
-  )
   (wire (pts (xy 45.72 101.6) (xy 52.07 101.6))
     (stroke (width 0) (type default))
@@
     (stroke (width 0) (type default))
   )
-  (wire (pts (xy 157.48 80.01) (xy 187.96 80.01))
+  (wire (pts (xy 149.86 80.01) (xy 187.96 80.01))
     (stroke (width 0) (type default))
   )
@@
     (stroke (width 0) (type default))
   )
-  (wire (pts (xy 157.48 72.39) (xy 157.48 80.01))
+  (wire (pts (xy 149.86 76.2) (xy 149.86 80.01))
     (stroke (width 0) (type default))
   )
@@
     )
   )
-  (symbol (lib_id "power:GND") (at 152.4 73.66 0) (unit 1)
-    (in_bom yes) (on_board yes) (dnp no)
-    (property "Reference" "#PWR011" (at 152.4 80.01 0)
-      (effects (font (size 1.27 1.27)) hide)
-    )
-    (property "Value" "GND" (at 152.4 77.47 0)
-      (effects (font (size 1.27 1.27)))
-    )
-    (property "Footprint" "" (at 152.4 73.66 0)
-      (effects (font (size 1.27 1.27)) hide)
-    )
-    (property "Datasheet" "" (at 152.4 73.66 0)
-      (effects (font (size 1.27 1.27)) hide)
-    )
-    (pin "1")
-    (instances
-      (project "UINIO-MCU-ESP32S3"
-        (path "/7b5dffae-532b-44bd-828e-e231478b308d"
-          (reference "#PWR011") (unit 1)
-        )
-      )
-    )
-  )
   (symbol (lib_id "Device:C") (at 44.45 35.56 0) (unit 1)
     (in_bom yes) (on_board yes) (dnp no)
@@
         (path "/7b5dffae-532b-44bd-828e-e231478b308d"
           (reference "#PWR027") (unit 1)
-        )
-      )
-    )
-  )
-  (symbol (lib_id "Device:Antenna_Chip") (at 154.94 69.85 0) (mirror y) (unit 1)
-    (in_bom yes) (on_board yes) (dnp no)
-    (property "Reference" "AE1" (at 150.495 61.595 0)
-      (effects (font (size 1.27 1.27)) (justify right))
-    )
-    (property "Value" "Antenna_Chip" (at 153.67 66.04 0)
-      (effects (font (size 1.27 1.27)) (justify right))
-    )
-    (property "Footprint" "RF_Antenna:Texas_SWRA117D_2.4GHz_Right" (at 157.48 65.405 0)
-      (effects (font (size 1.27 1.27)) hide)
-    )
-    (property "Datasheet" "~" (at 157.48 65.405 0)
-      (effects (font (size 1.27 1.27)) hide)
-    )
-    (pin "1")
-    (pin "2")
-    (instances
-      (project "UINIO-MCU-ESP32S3"
-        (path "/7b5dffae-532b-44bd-828e-e231478b308d"
-          (reference "AE1") (unit 1)
         )
       )
@@
         )
       )
+    )
+  )
+  (symbol (lib_id "Uinio:AN9520-245") (at 149.86 71.12 90) (unit 1)
+    (in_bom yes) (on_board yes) (dnp no)
+    (property "Reference" "L1" (at 144.78 71.12 90)
+      (effects (font (size 1.27 1.27)) (justify right))
+    )
+    (property "Value" "AN9520-245" (at 151.13 71.12 90)
+      (effects (font (size 1.27 1.27)) (justify right))
+    )
+    (property "Footprint" "Uinio:ANT-SMD_L9.5-W2.1" (at 151.3078 71.12 0)
+      (effects (font (size 1.27 1.27)) hide)
+    )
+    (property "Datasheet" "http://www.szlcsc.com/product/details_100880.html" (at 156.3878 71.12 0)
+      (effects (font (size 1.27 1.27)) hide)
+    )
+    (property "SuppliersPartNumber" "C99665" (at 161.4678 71.12 0)
+      (effects (font (size 1.27 1.27)) hide)
+    )
+    (property "uuid" "std:e4b513e4ba074533aff348d9b2e4d735" (at 161.4678 71.12 0)
+      (effects (font (size 1.27 1.27)) hide)
+    )
+    (pin "2")
+    (pin "1")
+    (instances
+      (project "UINIO-MCU-ESP32S3"
+        (path "/7b5dffae-532b-44bd-828e-e231478b308d"
+          (reference "L1") (unit 1)
+        )
+      )
